File: Tyr.sch (EAGLE design)
At the start: 210 parts, among them J1 TYR_DISPLAY, Q1 DTC123J, SW1 BUTTON, SW10 KEYSWITCH-MX-1U-HOTSWAP, SW11 KEYSWITCH-MX-1U-HOTSWAP, SW12 KEYSWITCH-MX-1U-HOTSWAP, SW13 KEYSWITCH-MX-1U-HOTSWAP, SW14 KEYSWITCH-MX-1U-HOTSWAP, SW15 KEYSWITCH-MX-1U-HOTSWAP, SW16 KEYSWITCH-MX-1U-HOTSWAP, SW17 KEYSWITCH-MX-1U-HOTSWAP, SW18 KEYSWITCH-MX-1U-HOTSWAP, SW19 KEYSWITCH-MX-1U-HOTSWAP, SW2 KEYSWITCH-MX-1U-HOTSWAP, SW20 KEYSWITCH-MX-1U-HOTSWAP, SW21 KEYSWITCH-MX-1U-HOTSWAP, SW22 KEYSWITCH-MX-1U-HOTSWAP, SW23 KEYSWITCH-MX-1U-HOTSWAP, SW24 KEYSWITCH-MX-1U-HOTSWAP, SW25 KEYSWITCH-MX-1U-HOTSWAPCAPSLO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, SW26 KEYSWITCH-MX-1U-HOTSWAP, SW27 KEYSWITCH-MX-1U-HOTSWAP, SW28 KEYSWITCH-MX-1U-HOTSWAP, SW29 KEYSWITCH-MX-1U-HOTSWAP, SW3 KEYSWITCH-MX-1U-HOTSWAP, SW30 KEYSWITCH-MX-1U-HOTSWAP, SW31 KEYSWITCH-MX-1U-HOTSWAP, SW32 KEYSWITCH-MX-2U-HOTSWAP, SW33 KEYSWITCH-MX-1U-HOTSWAP, SW34 KEYSWITCH-MX-1U-HOTSWAP, SW35 KEYSWITCH-MX-1U-HOTSWAP, SW36 KEYSWITCH-MX-1U-HOTSWAP, SW37 KEYSWITCH-MX-1U-HOTSWAP, SW38 KEYSWITCH-MX-1U-HOTSWAP, SW39 KEYSWITCH-MX-1U-HOTSWAP, SW4 KEYSWITCH-MX-1U-HOTSWAP, SW40 KEYSWITCH-MX-1U-HOTSWAP, SW41 KEYSWITCH-MX-2U-HOTSWAP, SW42 KEYSWITCH-MX-1U-HOTSWAP, SW5 KEYSWITCH-MX-1U-HOTSWAP, SW6 KEYSWITCH-MX-1U-HOTSWAP, SW7 KEYSWITCH-MX-1U-HOTSWAP, SW8 KEYSWITCH-MX-1U-HOTSWAP, SW9 KEYSWITCH-MX-1U-HOTSWAP, U1 MCP1700T, U2 PRTR5V0U2X, U3 STM32F303CC, U4 MB85RC256V, U6 TPS2552, X1 USB-C-12P-INBOARD, Y1 8Mhz

Commit message: Update
Parts:
- SW10, SW11, SW12, SW13, SW14, SW15, SW16, SW17, SW18, SW19, SW2, SW20, SW21, SW22, SW23, SW24, SW26, SW27, SW28, SW29, SW3, SW30, SW31, SW33, SW34, SW35, SW36, SW37, SW38, SW39, SW4, SW40, SW42, SW5, SW6, SW7, SW8, SW9: value KEYSWITCH-MX-1U-HOTSWAP -> KEYSWITCH-MX_PLATED-1U-HOTSWAP; device Tyr:KEYSWITCH-MX-1U-HOTSWAP -> Tyr:KEYSWITCH-MX_PLATED-1U-HOTSWAP
- SW25: value KEYSWITCH-MX-1U-HOTSWAPCAPSLOCK -> KEYSWITCH-MX_PLATED-1U-HOTSWAP_CAPSLOCK; device Tyr:KEYSWITCH-MX-1U-HOTSWAPCAPSLOCK -> Tyr:KEYSWITCH-MX_PLATED-1U-HOTSWAP_CAPSLOCK
- SW32, SW41: value KEYSWITCH-MX-2U-HOTSWAP -> KEYSWITCH-MX_PLATED-2U-HOTSWAP; device Tyr:KEYSWITCH-MX-2U-HOTSWAP -> Tyr:KEYSWITCH-MX_PLATED-2U-HOTSWAP

Commit message: Update
Changed lines of the file:
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@@
 </segment>
 <segment>
+<wire x1="281.94" y1="152.4" x2="281.94" y2="144.78" width="0.1524" layer="91"/>
+<pinref part="SUPPLY13" gate="GND" pin="GND"/>
 <pinref part="J1" gate="G$1" pin="3"/>
-<wire x1="299.72" y1="154.94" x2="281.94" y2="154.94" width="0.1524" layer="91"/>
-<wire x1="281.94" y1="154.94" x2="281.94" y2="144.78" width="0.1524" layer="91"/>
-<pinref part="SUPPLY13" gate="GND" pin="GND"/>
+<wire x1="299.72" y1="152.4" x2="281.94" y2="152.4" width="0.1524" layer="91"/>
 </segment>
 <segment>
@@
 </segment>
 <segment>
+<label x="284.48" y="162.56" size="1.27" layer="95" rot="R90" xref="yes"/>
 <pinref part="J1" gate="G$1" pin="4"/>
-<wire x1="299.72" y1="152.4" x2="284.48" y2="152.4" width="0.1524" layer="91"/>
-<wire x1="284.48" y1="152.4" x2="284.48" y2="162.56" width="0.1524" layer="91"/>
-<label x="284.48" y="162.56" size="1.27" layer="95" rot="R90" xref="yes"/>
-</segment>
-<segment>
+<wire x1="284.48" y1="154.94" x2="284.48" y2="162.56" width="0.1524" layer="91"/>
+<wire x1="299.72" y1="154.94" x2="284.48" y2="154.94" width="0.1524" layer="91"/>
+</segment>
+<segment>

Commit message: Rev0.5
Parts:
- C18, C19, C20, C21, C22, C23, C24, C25, C26, C27, C28, C29, C30, C31, C32, C33, C34, C35, C36, C37, C38, C39, C40, C41, C42, C43, C44, C45, C46, C47, C48, C49, C50, C51, C52: value 104 -> 100n
- HOLE1, HOLE2: value MOUNT_HOLE5MM_NOTCH -> MOUNT_HOLE-5MM_NOTCH; device Tyr:MOUNT_HOLE5MM_NOTCH -> Tyr:MOUNT_HOLE-5MM_NOTCH
- SW10, SW11, SW12, SW13, SW14, SW15, SW16, SW17, SW18, SW19, SW2, SW20, SW21, SW22, SW23, SW24, SW26, SW27, SW28, SW29, SW3, SW30, SW31, SW33, SW34, SW35, SW36, SW37, SW38, SW39, SW4, SW40, SW42, SW5, SW6, SW7, SW8, SW9: value KEYSWITCH-MX_PLATED-1U-HOTSWAP -> MX
- SW25: value KEYSWITCH-MX_PLATED-1U-HOTSWAP_CAPSLOCK -> MX
- SW32, SW41: value KEYSWITCH-MX_PLATED-2U-HOTSWAP -> MX

Commit message: Migrate to new library
Parts:
- C1, C10, C11, C12, C13, C14, C15, C16, C17, C18, C19, C2, C20, C21, C22, C23, C24, C25, C26, C27, C28, C29, C3, C30, C31, C32, C33, C34, C35, C36, C37, C38, C39, C4, C40, C41, C42, C43, C44, C45, C46, C47, C48, C49, C5, C50, C51, C52, C6, C7, C8, C9: device Tyr:CAPACITOR-0603 -> 1461748123:CAPACITOR-0603
- D1: device Tyr:DIODE_SCHOTTKY -> 1461748123:DIODE_SCHOTTKY
- D10, D11, D12, D13, D14, D15, D16, D17, D18, D19, D2, D20, D21, D22, D23, D24, D25, D26, D27, D28, D29, D3, D30, D31, D32, D33, D34, D35, D36, D37, D38, D39, D4, D40, D41, D42, D43, D44, D5, D6, D7, D8, D9: device Tyr:DIODE-SOD-123 -> 1461748123:DIODE-SOD-123
- HOLE1, HOLE2: device Tyr:MOUNT_HOLE-5MM_NOTCH -> 1461748123:MOUNT_HOLE-5MM_NOTCH
- HOLE3, HOLE4, HOLE5, HOLE6: device Tyr:MOUNT_HOLE -> 1461748123:MOUNT_HOLE
- J1: device Tyr:TYR_DISPLAY -> 1461748123:TYR_DISPLAY
- LED1, LED10, LED11, LED12, LED13, LED14, LED15, LED16, LED17, LED18, LED19, LED2, LED20, LED21, LED22, LED23, LED24, LED25, LED26, LED27, LED28, LED29, LED3, LED30, LED31, LED32, LED33, LED34, LED35, LED36, LED37, LED38, LED39, LED4, LED40, LED41, LED5, LED6, LED7, LED8, LED9: device Tyr:WS2812B_3528_REVERS-MOUNT -> 1461748123:WS2812B_3528_REVERS-MOUNT
- LOGO1: device Tyr:LOGO_TYR -> 1461748123:LOGO_TYR
- PH1: device Tyr:PINHEADER_1X6 -> 1461748123:PINHEADER_1X6
- Q1: device Tyr:DTC123J -> 1461748123:DTC123J
- R1, R11, R12, R2, R3, R4, R5, R6, R7, R8, R9: device Tyr:RESISTOR-0603 -> 1461748123:RESISTOR-0603
- R10: device Tyr:RESISTOR-2512 -> 1461748123:RESISTOR-2512
- SJ1: device Tyr:SOLDERJUMPER -> 1461748123:SOLDERJUMPER
- SW1: device Tyr:BUTTON -> 1461748123:BUTTON
- SW10, SW11, SW12, SW13, SW14, SW15, SW16, SW17, SW18, SW19, SW2, SW20, SW21, SW22, SW23, SW24, SW26, SW27, SW28, SW29, SW3, SW30, SW31, SW33, SW34, SW35, SW36, SW37, SW38, SW39, SW4, SW40, SW42, SW5, SW6, SW7, SW8, SW9: device Tyr:KEYSWITCH-MX_PLATED-1U-HOTSWAP -> 1461748123:KEYSWITCH-MX_PLATED-1U-HOTSWAP
- SW25: device Tyr:KEYSWITCH-MX_PLATED-1U-HOTSWAP_CAPSLOCK -> 1461748123:KEYSWITCH-MX_PLATED-1U-HOTSWAP_CAPSLOCK
- SW32, SW41: device Tyr:KEYSWITCH-MX_PLATED-2U-HOTSWAP -> 1461748123:KEYSWITCH-MX_PLATED-2U-HOTSWAP
- U1: device Tyr:MCP1700T -> 1461748123:MCP1700T
- U2: device Tyr:PRTR5V0U2X -> 1461748123:PRTR5V0U2X
- U3: device Tyr:STM32F303CC -> 1461748123:STM32F303CC
- U4: device Tyr:MB85RC256V -> 1461748123:MB85RC256V
- U5: device Tyr:INA219 -> 1461748123:INA219
- U6: device Tyr:TPS2552 -> 1461748123:TPS2552
- X1: device Tyr:CONTROLLER_USB-C-12PUSB-C-12P-INBOARD -> 1461748123:CONTROLLER_USB-C-12PUSB-C-12P-INBOARD
- Y1: device Tyr:CRYSTAL-4PIN-3.2X2.5 -> 1461748123:CRYSTAL-4PIN-3.2X2.5
